File: led_matrix.kicad_sch (KiCad schematic)
At the start: 0 parts

Commit message: Update KiCad project and schematic
Parts:
- added U1: XIAO-nRF52840-SMD, symbol seeed_xiao:XIAO-nRF52840-SMD
- added U2, U3: ~, Connector_ClipZin:299-008, symbol Connector:CLIP_Zin_8_Pin_299-008-299198
Connections:
- new net GND: U1.13 (GND), U1.16 (GND)

Commit message: Finished PCB
Parts:
- removed U2, U3: ~, Connector_ClipZin:299-008, symbol Connector:CLIP_Zin_8_Pin_299-008-299198
- added B1: S2B-PH-SM4-TB, jst:JST_S2B-PH-SM4-TB, symbol jst:S2B-PH-SM4-TB
- added C1, C2, C3: 22u, Capacitor_SMD:C_0805_2012Metric_Pad1.18x1.45mm_HandSolder, symbol Device:C
- added C10, C12: 0.1uF, Capacitor_SMD:C_0805_2012Metric_Pad1.18x1.45mm_HandSolder, symbol Device:C
- added C11: 1uF, Capacitor_SMD:C_0805_2012Metric_Pad1.18x1.45mm_HandSolder, symbol Device:C
- added C4, C9: 0.22u, Capacitor_Tantalum_SMD:CP_EIA-2012-15_AVX-P_HandSolder, symbol Device:C_Polarized_Small_US
- added C5: 8u, Capacitor_Tantalum_SMD:CP_EIA-2012-15_AVX-P_HandSolder, symbol Device:C_Polarized_Small_US
- added C6: 35p, Capacitor_SMD:C_0805_2012Metric_Pad1.18x1.45mm_HandSolder, symbol Device:C
- added C7: 10u, Capacitor_SMD:C_0805_2012Metric_Pad1.18x1.45mm_HandSolder, symbol Device:C
- added C8: 0.1u, Capacitor_SMD:C_0805_2012Metric_Pad1.18x1.45mm_HandSolder, symbol Device:C
- added J1, J2: Conn_01x07_Socket, Connector_PinSocket_2.54mm:PinSocket_1x07_P2.54mm_Vertical_SMD_Pin1Left, symbol Connector:Conn_01x07_Socket
- added J3: Conn_01x02_Pin, Connector_Wire:SolderWire-0.25sqmm_1x02_P4.5mm_D0.65mm_OD2mm, symbol Connector:Conn_01x02_Pin
- added J4: Conn_01x04_Pin, Connector_PinHeader_2.54mm:PinHeader_1x04_P2.54mm_Vertical_SMD_Pin1Left, symbol Connector:Conn_01x04_Pin
- added L1: 1u, Inductor_SMD:L_0805_2012Metric_Pad1.15x1.40mm_HandSolder, symbol Device:L
- added LED1, LED10, LED100, LED101, LED102, LED103, LED104, LED105, LED106, LED107, LED108, LED109, LED11, LED110, LED111, LED112, LED113, LED114, LED115, LED116, LED117, LED118, LED119, LED12, LED120, LED121, LED122, LED123, LED124, LED125, LED126, LED127, LED128, LED129, LED13, LED130, LED131, LED132, LED133, LED134, LED135, LED136, LED137, LED138, LED139, LED14, LED140, LED141, LED142, LED143, LED144, LED15, LED16, LED17, LED18, LED19, LED2, LED20, LED21, LED22, LED23, LED24, LED25, LED26, LED27, LED28, LED29, LED3, LED30, LED31, LED32, LED33, LED34, LED35, LED36, LED37, LED38, LED39, LED4, LED40, LED41, LED42, LED43, LED44, LED45, LED46, LED47, LED48, LED49, LED5, LED50, LED51, LED52, LED53, LED54, LED55, LED56, LED57, LED58, LED59, LED6, LED60, LED61, LED62, LED63, LED64, LED65, LED66, LED67, LED68, LED69, LED7, LED70, LED71, LED72, LED73, LED74, LED75, LED76, LED77, LED78, LED79, LED8, LED80, LED81, LED82, LED83, LED84, LED85, LED86, LED87, LED88, LED89, LED9, LED90, LED91, LED92, LED93, LED94, LED95, LED96, LED97, LED98, LED99: IN-S85AT5B, LED_IN-S85AT5B, symbol led:IN-S85AT5B
- added M1: CMA-4544PF-W, mic:MIC_CMA-4544PF-W, symbol mic:CMA-4544PF-W
- added R1: 4k, Resistor_SMD:R_0805_2012Metric_Pad1.20x1.40mm_HandSolder, symbol Device:R
- added R10, R8, R9: 4.7K, Resistor_SMD:R_0805_2012Metric_Pad1.20x1.40mm_HandSolder, symbol Device:R
- added R11: 20k, Resistor_SMD:R_0805_2012Metric_Pad1.20x1.40mm_HandSolder, symbol Device:R
- added R2, R3, R7: 100k, Resistor_SMD:R_0805_2012Metric_Pad1.20x1.40mm_HandSolder, symbol Device:R
- added R4: 10k, Resistor_SMD:R_0805_2012Metric_Pad1.20x1.40mm_HandSolder, symbol Device:R
- added R5: 34K, LED_SMD:LED_0805_2012Metric_Pad1.15x1.40mm_HandSolder, symbol Device:R
- added R6: 49.9, Resistor_SMD:R_0805_2012Metric_Pad1.20x1.40mm_HandSolder, symbol Device:R
- added U2: OPA1678IDR, opamp:SOIC127P599X175-8N, symbol opamp:OPA1678IDR
- added U3: TPS61235PRWLT, boost:CONV_TPS61235PRWLT, symbol boost:TPS61235PRWLT
- added U4: IS31FL3731-QF, led_driver:QFN40P400X400X80-29N-D, symbol Driver_LED:IS31FL3731-QF
- U1: footprint (none) -> seeed_xiao:custom_xiao_dip_pogo
Connections:
- net GND: now also U1.22 (GND), B1.2, C1.2, C10.2, C11.2, C12.2, C2.2, C3.2, C4.2, C7.2, C8.2, J2.6 (Pin_6), J4.4 (Pin_4), M1.2, R11.2, R3.2, R4.2, R7.2, U2.4 (V-), U3.1 (PGND), U3.4 (CC), U3.5 (AGND), U3.8 (INACT), U4.18 (AD), U4.29 (GND), U4.5 (GND)
- net A0: now reaches U1.1 (PA02_A0_D0)
- net A0: now also J1.1 (Pin_1)
- net D9: now reaches U1.10 (PA5_A9_D9_MISO)
- net D9: now also J2.3 (Pin_3)
- net D10: now reaches U1.11 (PA6_A10_D10_MOSI)
- net D10: now also J2.4 (Pin_4)
- net MCU_3_3V: now reaches U1.12 (3V3)
- net MCU_3_3V: now also J2.5 (Pin_5)
- net MCU_5V: now reaches U1.14 (5V)
- net MCU_5V: now also J2.7 (Pin_7)
- net +BATT: now reaches U1.15 (BAT)
- net +BATT: now also B1.1, C7.1, L1.1, L1.2, U3.2 (SW), U3.3 (VIN)
- net NF1_N: now reaches U1.17 (NFC1)
- net NF1_N: now also J3.2 (Pin_2)
- net NF1_P: now reaches U1.18 (NFC2)
- net NF1_P: now also J3.1 (Pin_1)
- net SWDIO: now reaches U1.19 (PA31_SWDIO)
- net SWDIO: now also J4.1 (Pin_1)
- net A1: now reaches U1.2 (PA4_A1_D1)
- net A1: now also J1.2 (Pin_2)
- net SWCLK: now reaches U1.20 (PA30_SWCLK)
- net SWCLK: now also J4.2 (Pin_2)
- net RESET: now reaches U1.21 (RESET)
- net RESET: now also J4.3 (Pin_3)
- net A2: now reaches U1.3 (PA10_A2_D2)
- net A2: now also J1.3 (Pin_3)
- net A3: now reaches U1.4 (PA11_A3_D3)
- net A3: now also J1.4 (Pin_4), R8.2, U4.4 (~{INTB})
- net A4: now reaches U1.5 (PA8_A4_D4_SDA)
- net A4: now also J1.5 (Pin_5), R10.2, U4.19 (SDA)
- net A5: now reaches U1.6 (PA9_A5_D5_SCL)
- net A5: now also J1.6 (Pin_6), R9.2, U4.20 (SCL)
- net D6: now reaches U1.7 (PB08_A6_D6_TX)
- net D6: now also J1.7 (Pin_7), R7.1, U4.3 (~{SDB})
- net D7: now reaches U1.8 (PB09_A7_D7_RX)
- net D7: now also J2.1 (Pin_1), R4.1, U3.7 (EN)
- net D8: now reaches U1.9 (PA7_A8_D8_SCK)
- net D8: now also J2.2 (Pin_2)
- new net: C10.1, U4.16 (C_FILT)
- new net: R11.1, U4.6 (R_EXT)
- new net: C4.1, R2.2, R3.1, U2.3 (+INA)
- new net: C5.1, C6.1, R5.1, U2.2 (-INA)
- new net: C6.2, R5.2, R6.2, U2.1 (OUTA)
- new net: C9.1, R6.1
- new net +5V: C1.1, C11.1, C12.1, C2.1, C3.1, C8.1, R1.1, R10.1, R2.1, R8.1, R9.1, U2.8 (V+), U3.6 (FB), U3.9 (VOUT), U4.2 (VCC)
- new net Audio_In: C9.2, U4.17 (IN)
- new net CA1_A: LED1.1, LED109.1, LED127.1, LED19.1, LED2.2, LED3.2, LED37.1, LED4.2, LED5.2, LED6.2, LED7.2, LED72.1, LED73.1, LED8.2, LED9.2, LED91.1, U4.21 (CA1)
- new net CA2_A: LED1.2, LED110.1, LED128.1, LED2.1, LED20.1, LED21.2, LED22.2, LED23.2, LED24.2, LED25.2, LED26.2, LED27.2, LED38.1, LED55.1, LED74.1, LED92.1, U4.22 (CA2)
- new net CA3_A: LED111.1, LED129.1, LED19.2, LED20.2, LED21.1, LED3.1, LED39.1, LED40.2, LED41.2, LED42.2, LED43.2, LED44.2, LED45.2, LED56.1, LED75.1, LED93.1, U4.23 (CA3)
- new net CA4_A: LED112.1, LED130.1, LED22.1, LED37.2, LED38.2, LED39.2, LED4.1, LED40.1, LED57.1, LED58.2, LED59.2, LED60.2, LED61.2, LED62.2, LED76.1, LED94.1, U4.24 (CA4)
- new net CA5_A: LED113.1, LED131.1, LED23.1, LED41.1, LED5.1, LED55.2, LED56.2, LED57.2, LED58.1, LED72.2, LED77.1, LED78.2, LED79.2, LED80.2, LED81.2, LED95.1, U4.25 (CA5)
- new net CA6_A: LED114.1, LED132.1, LED24.1, LED42.1, LED59.1, LED6.1, LED73.2, LED74.2, LED75.2, LED76.2, LED77.2, LED78.1, LED96.1, LED97.2, LED98.2, LED99.2, U4.26 (CA6)
- new net CA7_A: LED115.1, LED116.2, LED117.2, LED133.1, LED25.1, LED43.1, LED60.1, LED7.1, LED79.1, LED91.2, LED92.2, LED93.2, LED94.2, LED95.2, LED96.2, LED97.1, U4.27 (CA7)
- new net CA8_A: LED109.2, LED110.2, LED111.2, LED112.2, LED113.2, LED114.2, LED115.2, LED116.1, LED134.1, LED144.2, LED26.1, LED44.1, LED61.1, LED8.1, LED80.1, LED98.1, U4.28 (CA8)
- new net CA9_A: LED117.1, LED127.2, LED128.2, LED129.2, LED130.2, LED131.2, LED132.2, LED133.2, LED134.2, LED144.1, LED27.1, LED45.1, LED62.1, LED81.1, LED9.1, LED99.1, U4.1 (CA9)
- new net CB1_A: LED10.1, LED100.1, LED11.2, LED118.1, LED12.2, LED13.2, LED135.1, LED14.2, LED15.2, LED16.2, LED17.2, LED18.2, LED28.1, LED46.1, LED63.1, LED82.1, U4.7 (CB1)
- new net CB2_A: LED10.2, LED101.1, LED11.1, LED119.1, LED136.1, LED29.1, LED30.2, LED31.2, LED32.2, LED33.2, LED34.2, LED35.2, LED36.2, LED47.1, LED64.1, LED83.1, U4.8 (CB2)
- new net CB3_A: LED102.1, LED12.1, LED120.1, LED137.1, LED28.2, LED29.2, LED30.1, LED48.1, LED49.2, LED50.2, LED51.2, LED52.2, LED53.2, LED54.2, LED65.1, LED84.1, U4.9 (CB3)
- new net CB4_A: LED103.1, LED121.1, LED13.1, LED138.1, LED31.1, LED46.2, LED47.2, LED48.2, LED49.1, LED66.1, LED67.2, LED68.2, LED69.2, LED70.2, LED71.2, LED85.1, U4.10 (CB4)
- new net CB5_A: LED104.1, LED122.1, LED139.1, LED14.1, LED32.1, LED50.1, LED63.2, LED64.2, LED65.2, LED66.2, LED67.1, LED86.1, LED87.2, LED88.2, LED89.2, LED90.2, U4.11 (CB5)
- new net CB6_A: LED105.1, LED106.2, LED107.2, LED108.2, LED123.1, LED140.1, LED15.1, LED33.1, LED51.1, LED68.1, LED82.2, LED83.2, LED84.2, LED85.2, LED86.2, LED87.1, U4.12 (CB6)
- new net CB7_A: LED100.2, LED101.2, LED102.2, LED103.2, LED104.2, LED105.2, LED106.1, LED124.1, LED125.2, LED126.2, LED141.1, LED16.1, LED34.1, LED52.1, LED69.1, LED88.1, U4.13 (CB7)
- new net CB8_A: LED107.1, LED118.2, LED119.2, LED120.2, LED121.2, LED122.2, LED123.2, LED124.2, LED125.1, LED142.1, LED143.2, LED17.1, LED35.1, LED53.1, LED70.1, LED89.1, U4.14 (CB8)
- new net CB9_A: LED108.1, LED126.1, LED135.2, LED136.2, LED137.2, LED138.2, LED139.2, LED140.2, LED141.2, LED142.2, LED143.1, LED18.1, LED36.1, LED54.1, LED71.1, LED90.1, U4.15 (CB9)
- new net MIC: C5.2, M1.1, R1.2
- no-connect marks 0 -> 3
Other:
- note added: "5V Boost Converter"
- note added: "Connectors/Pin Header"
- note added: "LED Matrix"
- note added: "LED Matrix Drivers"
- note added: "Microcontroller"
- note added: "Single Supply Pre-Amp"
- moved on the sheet: U1
